Commit message: added model for rviz and gazebo

File: install/bumperbot_description/share/bumperbot_description/urdf/bumperbot.urdf.xacro (robot description, xacro)
@@ -3,4 +3,11 @@
     <link name="base_footprint"/>
     <link name="base_link">
+        <inertial>
+           <origin xyz="0 0 0.04" rpy="0.0 0.25 0.3" />
+           <mass value="8.2573504e-01"/>
+           <inertia ixx="2.2124416e-02" ixy="-1.2294101e-04" ixz="3.4938785e-04"
+               iyy="2.1193702e-02" iyz="-5.0120904e-05"
+               izz="2.0064271e-02" />
+        </inertial>
         <visual>
           <origin rpy="0 0 0" xyz="0 0 0"/>
@@ -9,4 +16,10 @@
           </geometry>
         </visual>
+        <collision>
+          <origin rpy="0 0 0" xyz="0 0 0"/>
+          <geometry>
+             <mesh filename="package://bumperbot_description/meshes/base_link.STL"/>
+          </geometry>
+        </collision>
     </link>
     <joint name="base_joint" type="fixed">
@@ -16,4 +29,11 @@
     </joint>
     <link name="wheel_right_link">
+        <inertial>
+            <origin xyz="0 -0.014 0" rpy="0 0 0" />
+            <mass value="0.0530086090966721" />
+            <inertia ixx="1.88176298336665E-05" ixy="-4.8444933029987E-10" ixz="1.88163708851143E-08"
+               iyy="3.11510738647764E-05" iyz="-6.93560663069607E-11"
+               izz="1.8801969558182E-05" />
+        </inertial>
         <visual>
            <origin rpy="1.57 0 0" xyz="0 0 0"/>
@@ -22,4 +42,10 @@
            </geometry>
         </visual>
+        <collision>
+            <origin xyz="0 -0.015 0" rpy="-1.57 0 0"/>
+            <geometry>
+               <sphere radius="0.033"/>
+            </geometry>
+        </collision>
     </link>
     <joint name="wheel_right_joint" type="continuous">
@@ -30,4 +56,11 @@
     </joint>
     <link name="wheel_left_link">
+        <inertial>
+            <origin xyz="0 0.014 0" rpy="0 0 0" />
+            <mass value="0.0530086043217644" />
+            <inertia ixx="1.8792911368909E-05"  ixy="3.31256392204584E-10" ixz="-1.14082001662767E-08"
+               iyy="3.11510738759073E-05" iyz="-3.60499245082192E-10"
+               izz="1.88266886146847E-05" />
+        </inertial>
         <visual>
            <origin rpy="-1.57 0 0" xyz="0 0 0"/>
@@ -36,4 +69,10 @@
            </geometry>
         </visual>
+        <collision>
+            <origin xyz="0 0.015 0" rpy="1.57 0 0"/>
+            <geometry>
+               <sphere radius="0.033"/>
+            </geometry>
+        </collision>
     </link>
     <joint name="wheel_left_joint" type="continuous">
@@ -44,4 +83,11 @@
     </joint>
     <link name="caster_front_wheel">
+        <inertial>
+            <origin xyz="3.89968128948481E-07 2.40073004698083E-07 0.00219173397061506" rpy="0 0 0" />
+            <mass value="1.44379265037903E-06" />
+            <inertia ixx="7.23075276010246E-11" ixy="-6.10956883467859E-16" ixz="2.22849693525031E-15"
+               iyy="3.8713793085917E-11"  iyz="2.93909858781952E-15"
+               izz="1.00967486676306E-10" />
+        </inertial>
         <visual>
            <origin rpy="0 0 0" xyz="0 0 0"/>
@@ -50,4 +96,10 @@
            </geometry>
         </visual>
+        <collision>
+            <origin xyz="0 0 0" rpy="0 0 0"/>
+            <geometry>
+               <sphere radius="0.005"/>
+            </geometry>
+        </collision>
     </link>
     <joint name="caster_front_joint" type="fixed">
@@ -58,4 +110,11 @@
     </joint>
     <link name="caster_rear_wheel">
+        <inertial>
+            <origin xyz="3.8996812895542E-07 2.40073004698083E-07 0.00219173397061509" rpy="0 0 0" />
+            <mass value="1.44379265037902E-06" />
+            <inertia ixx="7.23075276010246E-11" ixy="-6.10956872363424E-16" ixz="2.22849693527207E-15"
+               iyy="3.87137930859167E-11" iyz="2.939098587861E-15"
+               izz="1.00967486676306E-10" />
+        </inertial>
         <visual>
            <origin rpy="0 0 0" xyz="0 0 0"/>
@@ -64,4 +123,10 @@
            </geometry>
         </visual>
+        <collision>
+            <origin xyz="0 0 0" rpy="0 0 0"/>
+            <geometry>
+               <sphere radius="0.005"/>
+            </geometry>
+        </collision>
     </link>
     <joint name="caster_rear_joint" type="fixed">

Commit message: added simple velocity controller via ros2 control

File: install/bumperbot_description/share/bumperbot_description/urdf/bumperbot.urdf.xacro (robot description, xacro)
@@ -1,4 +1,6 @@
 <?xml version="1.0"?>
 <robot xmlns:xacro="http://www.ros.org/wiki/xacro" name="bumperbot">
+    <xacro:include filename="$(find bumperbot_description)/urdf/bumperbot_gazebo.xacro"/>
+    <xacro:include filename="$(find bumperbot_description)/urdf/bumperbot_ros2_control.xacro"/>
     <link name="base_footprint"/>
     <link name="base_link">

File: install/bumperbot_description/share/bumperbot_description/urdf/bumperbot_gazebo.xacro (robot description, xacro)
@@ -1,4 +1,24 @@
-<?xml version="1.0">
+<?xml version="1.0"?>
 <robot xmlns:xacro="http://www.ros.org/wiki/xacro" name="bumperbot">
+<!-- Right Wheel Transmission -->
+<transmission name="wheel_right_transmission">
+  <type>transmission_interface/SimpleTransmission</type>
+  <joint name="wheel_right_joint">
+    <hardwareInterface>hardware_interface/VelocityJointInterface</hardwareInterface>
+  </joint>
+  <actuator name="wheel_right_motor">
+    <mechanicalReduction>1.0</mechanicalReduction>
+  </actuator>
+</transmission>
+<!-- Left Wheel Transmission -->
+<transmission name="wheel_left_transmission">
+  <type>transmission_interface/SimpleTransmission</type>
+  <joint name="wheel_left_joint">
+    <hardwareInterface>hardware_interface/VelocityJointInterface</hardwareInterface>
+  </joint>
+  <actuator name="wheel_left_motor">
+    <mechanicalReduction>1.0</mechanicalReduction>
+  </actuator>
+</transmission>
   <!-- Wheels -->
   <gazebo reference="wheel_left_link">
@@ -37,3 +57,10 @@
     <maxVel>1.0</maxVel>
   </gazebo>
+  <gazebo>
+      <plugin filename="libgazebo_ros2_control.so" name="gazebo_ros2_control">
+          <robot_param>robot_description</robot_param>
+          <robot_param_node>robot_state_publisher</robot_param_node>
+          <parameters>/home/aakash/bumperbot_ws/src/bumperbot_controller/config/bumperbot_controllers.yaml</parameters>
+      </plugin>
+  </gazebo>
 </robot>

File: src/bumperbot_description/urdf/bumperbot_gazebo.xacro (robot description, xacro)
@@ -1,4 +1,24 @@
-<?xml version="1.0">
+<?xml version="1.0"?>
 <robot xmlns:xacro="http://www.ros.org/wiki/xacro" name="bumperbot">
+<!-- Right Wheel Transmission -->
+<transmission name="wheel_right_transmission">
+  <type>transmission_interface/SimpleTransmission</type>
+  <joint name="wheel_right_joint">
+    <hardwareInterface>hardware_interface/VelocityJointInterface</hardwareInterface>
+  </joint>
+  <actuator name="wheel_right_motor">
+    <mechanicalReduction>1.0</mechanicalReduction>
+  </actuator>
+</transmission>
+<!-- Left Wheel Transmission -->
+<transmission name="wheel_left_transmission">
+  <type>transmission_interface/SimpleTransmission</type>
+  <joint name="wheel_left_joint">
+    <hardwareInterface>hardware_interface/VelocityJointInterface</hardwareInterface>
+  </joint>
+  <actuator name="wheel_left_motor">
+    <mechanicalReduction>1.0</mechanicalReduction>
+  </actuator>
+</transmission>
   <!-- Wheels -->
   <gazebo reference="wheel_left_link">
@@ -37,3 +57,10 @@
     <maxVel>1.0</maxVel>
   </gazebo>
+  <gazebo>
+      <plugin filename="libgazebo_ros2_control.so" name="gazebo_ros2_control">
+          <robot_param>robot_description</robot_param>
+          <robot_param_node>robot_state_publisher</robot_param_node>
+          <parameters>/home/aakash/bumperbot_ws/src/bumperbot_controller/config/bumperbot_controllers.yaml</parameters>
+      </plugin>
+  </gazebo>
 </robot>
